File: Breadboard_Power_Supply.kicad_sch (KiCad schematic)
At the start: 17 parts, among them J1 Conn_01x02_Pin, J2 Conn_01x02_Pin, J3 Conn_01x03_Pin, J4 Conn_01x03_Pin, J5 Screw_Terminal_01x02, J6 Barrel_Jack_Switch, J7 Screw_Terminal_01x02, SW1 SW_Wuerth_450301014042, U1 LM7805_TO220, U2 LM317_TO-220

Commit message: Complete PCB layout and add manufacturing files
Connections:
- net PWR_Output renamed PWR_OUT_BOTTON
- net PWR_OUT_BOTTON: no longer J1.2 (Pin_2), J3.2 (Pin_2), J7.2 (Pin_2)
- new net PWR_OUT_TOP: J1.2 (Pin_2), J3.2 (Pin_2), J7.2 (Pin_2)
Changed lines of the file:
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@@
+		)
+	)
+	(label "PWR_OUT_BOTTON"
+		(at 205.74 123.19 0)
+		(effects
+			(font
+				(size 1.27 1.27)
+			)
+			(justify left bottom)
 		)
 	)
@@
 		)
 	)
-	(label "PWR_Output"
-		(at 205.74 121.92 0)
-		(effects
-			(font
-				(size 1.27 1.27)
-			)
-			(justify left bottom)
-		)
-	)
-	(label "PWR_Output"
+	(label "PWR_OUT_TOP"
 		(at 208.28 60.96 0)
 		(effects
