File: Breadboard_Power_Supply.kicad_pcb (KiCad board)
At the start: 2 copper layers, 31 x 53.1 mm, 17 parts, among them J1 Conn_01x02_Pin, J2 Conn_01x02_Pin, J3 Conn_01x03_Pin, J4 Conn_01x03_Pin, J5 Screw_Terminal_01x02, J6 Barrel_Jack_Switch, J7 Screw_Terminal_01x02, SW1 SW_Wuerth_450301014042, U1 LM7805_TO220, U2 LM317_TO-220

Commit message: Fix component position on PCB
Parts:
- moved J7 5.74 mm to (70.7, 39.3), turned to 180 degrees
Routing:
- net /PWR_OUT_TOP: track 23.1 -> 25.8 mm
Changed lines of the file:
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@@
 	(footprint "TerminalBlock_Phoenix:TerminalBlock_Phoenix_MKDS-1,5-2-5.08_1x02_P5.08mm_Horizontal"
 		(layer "F.Cu")
-		(at 65.019 39.8473)
+		(at 70.739 39.3446 180)
 		(descr "Terminal Block Phoenix MKDS-1,5-2-5.08, 2 pins, pitch 5.08mm, size 10.2x9.8mm, drill diameter 1.3mm, pad diameter 2.6mm, http://www.farnell.com/datasheets/100425.pdf, script-generated using https://gitlab.com/kicad/libraries/kicad-footprint-generator/-/tree/master/scripts/TerminalBlock_Phoenix")
 		(tags "THT Terminal Block Phoenix MKDS-1,5-2-5.08 pitch 5.08mm size 10.2x9.8mm drill 1.3mm pad 2.6mm")
@@
 		(attr through_hole)
 		(fp_line
-			(start -2.66 -5.32)
-			(end 7.74 -5.32)
+			(start 7.74 4.72)
+			(end 0.3 4.72)
 			(stroke
 				(width 0.12)
@@
 		)
 		(fp_line
-			(start -2.66 -2.3)
-			(end 7.74 -2.3)
+			(start 7.74 -5.32)
+			(end 7.74 4.72)
 			(stroke
 				(width 0.12)
@@
 		)
 		(fp_line
-			(start -2.66 2.6)
-			(end 7.74 2.6)
+			(start -0.3 4.72)
+			(end -2.66 4.72)
 			(stroke
 				(width 0.12)
@@
 		)
 		(fp_line
-			(start -2.66 4.1)
-			(end 7.74 4.1)
+			(start -2.66 4.72)
+			(end -2.66 -5.32)
 			(stroke
 				(width 0.12)
@@
 		)
 		(fp_line
-			(start -2.66 4.72)
-			(end -2.66 -5.32)
+			(start -2.66 4.1)
+			(end 7.74 4.1)
 			(stroke
 				(width 0.12)
@@
 		)
 		(fp_line
-			(start -0.3 4.72)
-			(end -2.66 4.72)
+			(start -2.66 2.6)
+			(end 7.74 2.6)
 			(stroke
 				(width 0.12)
@@
 		)
 		(fp_line
-			(start 7.74 -5.32)
-			(end 7.74 4.72)
+			(start -2.66 -2.3)
+			(end 7.74 -2.3)
 			(stroke
 				(width 0.12)
@@
 		)
 		(fp_line
-			(start 7.74 4.72)
-			(end 0.3 4.72)
+			(start -2.66 -5.32)
+			(end 7.74 -5.32)
 			(stroke
 				(width 0.12)
@@
 		)
 		(fp_line
-			(start -3.04 -5.71)
-			(end -3.04 5.1)
+			(start 8.13 5.1)
+			(end 8.13 -5.71)
 			(stroke
 				(width 0.05)
@@
 		)
 		(fp_line
-			(start -3.04 5.1)
-			(end 8.13 5.1)
+			(start 8.13 -5.71)
+			(end -3.04 -5.71)
 			(stroke
 				(width 0.05)
@@
 		)
 		(fp_line
-			(start 8.13 -5.71)
-			(end -3.04 -5.71)
+			(start -3.04 5.1)
+			(end 8.13 5.1)
 			(stroke
 				(width 0.05)
@@
 		)
 		(fp_line
-			(start 8.13 5.1)
-			(end 8.13 -5.71)
+			(start -3.04 -5.71)
+			(end -3.04 5.1)
 			(stroke
 				(width 0.05)
@@
 		)
 		(fp_line
-			(start -2.54 -5.2)
-			(end 7.62 -5.2)
+			(start 7.62 4.6)
+			(end -2.04 4.6)
 			(stroke
 				(width 0.1)
@@
 		)
 		(fp_line
-			(start -2.54 -2.3)
-			(end 7.62 -2.3)
+			(start 7.62 -5.2)
+			(end 7.62 4.6)
 			(stroke
 				(width 0.1)
@@
 		)
 		(fp_line
-			(start -2.54 2.6)
-			(end 7.62 2.6)
+			(start 6.218 -0.955)
+			(end 4.125 1.138)
 			(stroke
 				(width 0.1)
@@
 		)
 		(fp_line
-			(start -2.54 4.1)
-			(end -2.54 -5.2)
+			(start 6.035 -1.138)
+			(end 3.942 0.955)
 			(stroke
 				(width 0.1)
@@
 		)
 		(fp_line
-			(start -2.54 4.1)
-			(end 7.62 4.1)
+			(start 1.138 -0.955)
+			(end -0.955 1.138)
 			(stroke
 				(width 0.1)
@@
 		)
 		(fp_line
-			(start -2.04 4.6)
-			(end -2.54 4.1)
+			(start 0.955 -1.138)
+			(end -1.138 0.955)
 			(stroke
 				(width 0.1)
@@
 		)
 		(fp_line
-			(start 0.955 -1.138)
-			(end -1.138 0.955)
+			(start -2.04 4.6)
+			(end -2.54 4.1)
 			(stroke
 				(width 0.1)
@@
 		)
 		(fp_line
-			(start 1.138 -0.955)
-			(end -0.955 1.138)
+			(start -2.54 4.1)
+			(end 7.62 4.1)
 			(stroke
 				(width 0.1)
@@
 		)
 		(fp_line
-			(start 6.035 -1.138)
-			(end 3.942 0.955)
+			(start -2.54 4.1)
+			(end -2.54 -5.2)
 			(stroke
 				(width 0.1)
@@
 		)
 		(fp_line
-			(start 6.218 -0.955)
-			(end 4.125 1.138)
+			(start -2.54 2.6)
+			(end 7.62 2.6)
 			(stroke
 				(width 0.1)
@@
 		)
 		(fp_line
-			(start 7.62 -5.2)
-			(end 7.62 4.6)
+			(start -2.54 -2.3)
+			(end 7.62 -2.3)
 			(stroke
 				(width 0.1)
@@
 		)
 		(fp_line
-			(start 7.62 4.6)
-			(end -2.04 4.6)
+			(start -2.54 -5.2)
+			(end 7.62 -5.2)
 			(stroke
 				(width 0.1)
@@
 		)
 		(fp_circle
-			(center 0 0)
-			(end 1.5 0)
+			(center 5.08 0)
+			(end 6.58 0)
 			(stroke
 				(width 0.1)
@@
 		)
 		(fp_circle
-			(center 5.08 0)
-			(end 6.58 0)
+			(center 0 0)
+			(end 1.5 0)
 			(stroke
 				(width 0.1)
@@
 		)
 		(pad "1" thru_hole roundrect
-			(at 0 0)
+			(at 0 0 180)
 			(size 2.6 2.6)
 			(drill 1.3)
@@
 		)
 		(pad "2" thru_hole circle
-			(at 5.08 0)
+			(at 5.08 0 180)
 			(size 2.6 2.6)
 			(drill 1.3)
@@
 	)
 	(gr_text "GND\n"
-		(at 62.359 46.355 0)
+		(at 69.469 46.228 0)
 		(layer "F.SilkS")
 		(effects
@@
 	)
 	(segment
-		(start 70.099 39.8473)
-		(end 65.0232 34.7715)
+		(start 65.659 39.3446)
+		(end 65.659 35.4073)
 		(width 0.3)
 		(layer "F.Cu")
@@
 	)
 	(segment
+		(start 76.962 38.608)
+		(end 75.9976 37.6436)
+		(width 0.3)
+		(layer "F.Cu")
+		(net 9)
+	)
+	(segment
 		(start 58.2232 34.7715)
 		(end 56.9722 36.0225)
@@
 	)
 	(segment
-		(start 75.7227 39.8473)
-		(end 70.099 39.8473)
+		(start 65.659 35.4073)
+		(end 65.0232 34.7715)
 		(width 0.3)
 		(layer "F.Cu")
@@
 	)
 	(segment
-		(start 76.962 38.608)
-		(end 75.7227 39.8473)
+		(start 75.9976 37.6436)
+		(end 67.36 37.6436)
+		(width 0.3)
+		(layer "F.Cu")
+		(net 9)
+	)
+	(segment
+		(start 67.36 37.6436)
+		(end 65.659 39.3446)
 		(width 0.3)
 		(layer "F.Cu")
